Commit message: Package name tweaks

File: kaia_description/urdf/kaia_snoopy.urdf (robot description, URDF)
Before this commit: robot kaia_waffle_pi, 11 links, 10 joints
Links:
- removed link camera_link
- removed link camera_rgb_frame
- removed link camera_rgb_optical_frame
- removed link caster_back_left_link
- removed link caster_back_right_link
- added link caster_back_link, mass 0.005; collision box size=0.030 0.009 0.020
- link base_link: mass 1.3729096e+00 -> 8.2573504e-01; geometry collision box size=0.140 0.140 0.143; visual mesh filename=package://kaia_description/meshes/bases/snoopy_base.stl scale=0.001 0.001 0.001
- link base_scan: geometry collision cylinder length=0.0315 radius=0.055; visual mesh filename=package://kaia_description/meshes/sensors/lds.stl scale=0.001 0.001 0.001
- link wheel_left_link: geometry collision cylinder length=0.018 radius=0.033; visual mesh filename=package://kaia_description/meshes/wheels/left_tire.stl scale=0.001 0.001 0.001
- link wheel_right_link: geometry collision cylinder length=0.018 radius=0.033; visual mesh filename=package://kaia_description/meshes/wheels/right_tire.stl scale=0.001 0.001 0.001
Joints:
- removed joint camera_joint
- removed joint camera_rgb_joint
- removed joint camera_rgb_optical_joint
- removed joint caster_back_left_joint
- removed joint caster_back_right_joint
- added joint caster_back_joint: type fixed, parent base_link, child caster_back_link, origin xyz=-0.081 0 -0.004 rpy=-1.57 0 0
- joint base_joint: origin xyz=0 0 0.010 rpy=0 0 0 -> xyz=0.0 0.0 0.010 rpy=0 0 0
- joint imu_joint: origin xyz=0.0 0 0.068 rpy=0 0 0 -> xyz=-0.032 0 0.068 rpy=0 0 0
- joint scan_joint: origin xyz=-0.064 0 0.122 rpy=0 0 0 -> xyz=-0.032 0 0.172 rpy=0 0 0
- joint wheel_left_joint: origin xyz=0.0 0.144 0.023 rpy=-1.57 0 0 -> xyz=0.0 0.08 0.023 rpy=-1.57 0 0
- joint wheel_right_joint: origin xyz=0.0 -0.144 0.023 rpy=-1.57 0 0 -> xyz=0.0 -0.080 0.023 rpy=-1.57 0 0
