Commit message: Rviz2 launch per model, package

File: kaia_description/urdf/goofy.urdf (robot description, URDF)
Before this commit: robot kaia_waffle, 13 links, 12 joints
Links:
- removed link camera_depth_frame
- removed link camera_depth_optical_frame
- link base_link: geometry collision box size=0.266 0.266 0.094; visual mesh filename=package://kaia_description/meshes/bases/goofy_base.stl scale=0.001 0.001 0.001
- link base_scan: geometry collision cylinder length=0.0315 radius=0.055; visual mesh filename=package://kaia_description/meshes/sensors/lds.stl scale=0.001 0.001 0.001
- link camera_link: geometry collision box size=0.015 0.030 0.027
- link wheel_left_link: geometry collision cylinder length=0.018 radius=0.033; visual mesh filename=package://kaia_description/meshes/wheels/left_tire.stl scale=0.001 0.001 0.001
- link wheel_right_link: geometry collision cylinder length=0.018 radius=0.033; visual mesh filename=package://kaia_description/meshes/wheels/right_tire.stl scale=0.001 0.001 0.001
Joints:
- removed joint camera_depth_joint
- removed joint camera_depth_optical_joint
- joint camera_joint: origin xyz=0.064 -0.065 0.094 rpy=0 0 0 -> xyz=0.073 -0.011 0.084 rpy=0 0 0
- joint camera_rgb_joint: origin xyz=0.005 0.018 0.013 rpy=0 0 0 -> xyz=0.003 0.011 0.009 rpy=0 0 0

File: kaia_description/urdf/loki.urdf (robot description, URDF)
Before this commit: robot kaia_waffle_pi, 11 links, 10 joints
Links:
- added link camera_depth_frame
- added link camera_depth_optical_frame
- link base_link: geometry collision box size=0.266 0.266 0.094; visual mesh filename=package://kaia_description/meshes/bases/loki_base.stl scale=0.001 0.001 0.001
- link camera_link: geometry collision box size=0.012 0.132 0.020; visual mesh filename=package://kaia_description/meshes/sensors/r200.dae
Joints:
- added joint camera_depth_joint: type fixed, parent camera_link, child camera_depth_frame, origin xyz=0.005 0.028 0.013 rpy=0 0 0
- added joint camera_depth_optical_joint: type fixed, parent camera_depth_frame, child camera_depth_optical_frame, origin xyz=0 0 0 rpy=-1.57 0 -1.57
- joint camera_joint: origin xyz=0.073 -0.011 0.084 rpy=0 0 0 -> xyz=0.064 -0.065 0.094 rpy=0 0 0
- joint camera_rgb_joint: origin xyz=0.003 0.011 0.009 rpy=0 0 0 -> xyz=0.005 0.018 0.013 rpy=0 0 0
